File: standard_power_supply/standard_power_supply.kicad_pcb (KiCad board)
At the start: 2 copper layers, 100 x 80 mm, 9 parts, among them J1 Conn_01x03, J4 +40V 0 -40V

Commit message: Resolve 90 degree copper connection.
Routing:
- net Net-(J1-Pin_2): track 99.2 -> 103.6 mm
Changed lines of the file:
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@@
 	)
 	(segment
-		(start 128.5 100)
-		(end 128.5 92.5)
+		(start 145 76)
+		(end 137.5 76)
+		(width 3)
+		(layer "B.Cu")
+		(net 2)
+	)
+	(segment
+		(start 137.5 76)
+		(end 128.5 85)
 		(width 3)
 		(layer "B.Cu")
@@
 	)
 	(segment
-		(start 161.5 92.5)
-		(end 145 76)
+		(start 128.5 85)
+		(end 128.5 100)
 		(width 3)
 		(layer "B.Cu")
@@
 	)
 	(segment
-		(start 128.5 92.5)
+		(start 161.5 92.5)
 		(end 145 76)
 		(width 3)
